File: schematics/ECG/Logic/ECG_Logic.sch (EAGLE design)
At the start: 78 parts, among them IC1 ADS1293, IC2 LIS3DH, IC3 MCP1703, IC4 CC2541, IC5 FSA4157, IC6 FSA4157, IC7 FSA4157, IC8 BALUN_2450BM_SERIES_SMD, P1 TARGET_RA, P2 TARGET_RA, P3 TARGET_RA, P4 TARGET_RA, P5 TARGET_RA, P6 TARGET_RA, P7 TARGET_RA, X1 XTAL-2SMD, X2 XTAL_403, X3 ECS-40-20-4VX

Commit message: RGB LED wiring was incorrect due to error in package. Using updated RGB LED package with correct wiring
Connections:
- net BLUE_LED: now also IC4.P1_7, R9.2; no longer IC4.P2_0, R8.2
- net RED_LED: now also IC4.P2_0, R8.2; no longer IC4.P1_7, R9.2
Changed lines of the file:
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@@
 <?xml version="1.0" encoding="utf-8"?>
 <!DOCTYPE eagle SYSTEM "eagle.dtd">
-<eagle version="6.4">
+<eagle version="6.5.0">
 <drawing>
 <settings>
@@
 </segment>
 </net>
-<net name="BLUE_LED" class="0">
+<net name="GREEN_LED" class="0">
+<segment>
+<pinref part="IC4" gate="G$1" pin="P1_6"/>
+<wire x1="243.84" y1="116.84" x2="248.92" y2="116.84" width="0.1524" layer="91"/>
+<junction x="243.84" y="116.84"/>
+<label x="248.92" y="116.84" size="1.27" layer="95"/>
+</segment>
+<segment>
+<pinref part="R31" gate="G$1" pin="2"/>
+<wire x1="228.6" y1="190.5" x2="231.14" y2="190.5" width="0.1524" layer="91"/>
+<junction x="228.6" y="190.5"/>
+<label x="231.14" y="190.5" size="1.27" layer="95"/>
+</segment>
+</net>
+<net name="N$3" class="0">
+<segment>
+<pinref part="TRI_LED" gate="LED" pin="B"/>
+<junction x="218.44" y="195.58"/>
+<pinref part="R9" gate="G$1" pin="1"/>
+</segment>
+</net>
+<net name="N$9" class="0">
+<segment>
+<pinref part="TRI_LED" gate="LED" pin="G"/>
+<junction x="218.44" y="190.5"/>
+<pinref part="R31" gate="G$1" pin="1"/>
+</segment>
+</net>
+<net name="N$20" class="0">
+<segment>
+<pinref part="TRI_LED" gate="LED" pin="R"/>
+<junction x="218.44" y="185.42"/>
+<pinref part="R8" gate="G$1" pin="1"/>
+</segment>
+</net>
+<net name="RED_LED" class="0">
 <segment>
 <pinref part="IC4" gate="G$1" pin="P2_0"/>
@@
 <junction x="228.6" y="185.42"/>
 <label x="231.14" y="185.42" size="1.27" layer="95"/>
-</segment>
-</net>
-<net name="GREEN_LED" class="0">
-<segment>
-<pinref part="IC4" gate="G$1" pin="P1_6"/>
-<wire x1="243.84" y1="116.84" x2="248.92" y2="116.84" width="0.1524" layer="91"/>
-<junction x="243.84" y="116.84"/>
-<label x="248.92" y="116.84" size="1.27" layer="95"/>
-</segment>
-<segment>
-<pinref part="R31" gate="G$1" pin="2"/>
-<wire x1="228.6" y1="190.5" x2="231.14" y2="190.5" width="0.1524" layer="91"/>
-<junction x="228.6" y="190.5"/>
-<label x="231.14" y="190.5" size="1.27" layer="95"/>
-</segment>
-</net>
-<net name="N$3" class="0">
-<segment>
-<pinref part="TRI_LED" gate="LED" pin="B"/>
-<junction x="218.44" y="195.58"/>
-<pinref part="R9" gate="G$1" pin="1"/>
-</segment>
-</net>
-<net name="N$9" class="0">
-<segment>
-<pinref part="TRI_LED" gate="LED" pin="G"/>
-<junction x="218.44" y="190.5"/>
-<pinref part="R31" gate="G$1" pin="1"/>
-</segment>
-</net>
-<net name="N$20" class="0">
-<segment>
-<pinref part="TRI_LED" gate="LED" pin="R"/>
-<junction x="218.44" y="185.42"/>
-<pinref part="R8" gate="G$1" pin="1"/>
-</segment>
-</net>
-<net name="RED_LED" class="0">
-<segment>
-<pinref part="R9" gate="G$1" pin="2"/>
-<wire x1="228.6" y1="195.58" x2="231.14" y2="195.58" width="0.1524" layer="91"/>
-<junction x="228.6" y="195.58"/>
-<label x="231.14" y="195.58" size="1.27" layer="95"/>
-</segment>
-<segment>
-<pinref part="IC4" gate="G$1" pin="P1_7"/>
-<wire x1="243.84" y1="119.38" x2="248.92" y2="119.38" width="0.1524" layer="91"/>
-<junction x="243.84" y="119.38"/>
-<label x="248.92" y="119.38" size="1.27" layer="95"/>
 </segment>
 </net>
@@
 </segment>
 </net>
+<net name="BLUE_LED" class="0">
+<segment>
+<pinref part="IC4" gate="G$1" pin="P1_7"/>
+<wire x1="243.84" y1="119.38" x2="248.92" y2="119.38" width="0.1524" layer="91"/>
+<junction x="243.84" y="119.38"/>
+<label x="248.92" y="119.38" size="1.27" layer="95"/>
+</segment>
+<segment>
+<pinref part="R9" gate="G$1" pin="2"/>
+<wire x1="228.6" y1="195.58" x2="231.14" y2="195.58" width="0.1524" layer="91"/>
+<junction x="228.6" y="195.58"/>
+<label x="231.14" y="195.58" size="1.27" layer="95"/>
+</segment>
+</net>
