File: schematics/ECG/Patch/ECG_Patch.brd (EAGLE design)
At the start: 11.6 x 27.7 mm, 10 parts

Commit message: fixed charger board piston naming
Parts:
- renumbered U$1 to P2, U$2 to P3, U$3 to P4, U$4 to P5, U$5 to P1, U$6 to P6
Changed lines of the file:
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@@
 </autorouter>
 <elements>
-<element name="U$1" library="pins" package="PISTON_RA_TH" value="PISTON_RA_TH" x="2.54" y="16.002" rot="R180"/>
-<element name="U$2" library="pins" package="PISTON_RA_TH" value="PISTON_RA_TH" x="2.54" y="13.462" rot="R180"/>
-<element name="U$3" library="pins" package="PISTON_RA_TH" value="PISTON_RA_TH" x="2.54" y="10.922" rot="R180"/>
-<element name="U$4" library="pins" package="PISTON_RA_TH" value="PISTON_RA_TH" x="2.54" y="8.382" rot="R180"/>
-<element name="U$5" library="pins" package="PISTON_RA_TH" value="PISTON_RA_TH" x="2.54" y="25.781" rot="R180"/>
-<element name="U$6" library="pins" package="PISTON_RA_TH" value="PISTON_RA_TH" x="2.54" y="1.905" rot="R180"/>
+<element name="P2" library="pins" package="PISTON_RA_TH" value="PISTON_RA_TH" x="2.54" y="16.002" rot="R180"/>
+<element name="P3" library="pins" package="PISTON_RA_TH" value="PISTON_RA_TH" x="2.54" y="13.462" rot="R180"/>
+<element name="P4" library="pins" package="PISTON_RA_TH" value="PISTON_RA_TH" x="2.54" y="10.922" rot="R180"/>
+<element name="P5" library="pins" package="PISTON_RA_TH" value="PISTON_RA_TH" x="2.54" y="8.382" rot="R180"/>
+<element name="P1" library="pins" package="PISTON_RA_TH" value="PISTON_RA_TH" x="2.54" y="25.781" rot="R180"/>
+<element name="P6" library="pins" package="PISTON_RA_TH" value="PISTON_RA_TH" x="2.54" y="1.905" rot="R180"/>
 <element name="LL" library="wirepad" package="1,6/0,8" value="" x="10.414" y="13.462"/>
 <element name="RL" library="wirepad" package="1,6/0,8" value="" x="10.414" y="16.002"/>
@@
 <signals>
 <signal name="LL">
-<contactref element="U$2" pad="1"/>
+<contactref element="P3" pad="1"/>
 <contactref element="LL" pad="1"/>
 <wire x1="7.874" y1="13.462" x2="10.414" y2="13.462" width="0.4064" layer="1"/>
 </signal>
 <signal name="RL">
-<contactref element="U$1" pad="1"/>
+<contactref element="P2" pad="1"/>
 <contactref element="RL" pad="1"/>
 <wire x1="7.874" y1="16.002" x2="10.414" y2="16.002" width="0.4064" layer="1"/>
 </signal>
 <signal name="LA">
-<contactref element="U$3" pad="1"/>
+<contactref element="P4" pad="1"/>
 <contactref element="LA" pad="1"/>
 <wire x1="7.874" y1="10.922" x2="10.414" y2="10.922" width="0.4064" layer="1"/>
 </signal>
 <signal name="RA">
-<contactref element="U$4" pad="1"/>
+<contactref element="P5" pad="1"/>
 <contactref element="RA" pad="1"/>
 <wire x1="7.874" y1="8.382" x2="10.414" y2="8.382" width="0.4064" layer="1"/>
 </signal>
 <signal name="BATT">
-<contactref element="U$5" pad="1"/>
-<contactref element="U$6" pad="1"/>
+<contactref element="P1" pad="1"/>
+<contactref element="P6" pad="1"/>
 <wire x1="1.4224" y1="5.7912" x2="1.4224" y2="19.812" width="0.4064" layer="1"/>
 <wire x1="7.874" y1="1.905" x2="7.874" y2="3.2512" width="0.4064" layer="1"/>
